File: hat.sch (EAGLE design)
At the start: 13 parts, among them U1 HEX_CONVERTER

Commit message: Work in progess
Parts:
- added IC1: 24LC-I/OT, we-chip:24LC-I/OT
- added LED1: RED, led:LEDCHIPLED_0805
- added R2, R3, R5: 3k9, resistor:R-EU_R0805
- added R4: 330, rcl:R-EU_R0805
- added SJ1: (no value), jumper:SJ
- C1, C2: value (none) -> 15p
- C3: value (none) -> 100n
- Q1: value (none) -> 12mHz
- R1: value (none) -> 10k; device SparkFun-Resistors:RESISTOR1206 -> resistor:R-EU_R0805
Connections:
- new net ID_SC: IC1.SCL, R2.1, RPI1.ID_SC
- new net ID_SD: IC1.SDA, R5.2, RPI1.ID_SD
- new net N$5: IC1.WP, R3.1, SJ1.2
- new net N$7: LED1.A, RPI1.IO17
- new net N$8: LED1.C, R4.1
- net GND: now also IC1.GND, R4.2, SJ1.1; no longer RPI1.GND@1, RPI1.GND@3
- net VCC: now also IC1.VCC, R2.2, R3.2, R5.1
Other:
- moved on the sheet: C1, C2, C3, Q1, RPI1, SV1, SV2, SV3, SV4, SV5, U$1, U1

Commit message: Add board
Connections:
- removed net USCK: U$1.(PCINT4/T1/SCL/USCK/ADC4)PA4
- new net +5V: RPI1.5V@1, SV2.2, SV3.2, SV4.2, SV5.2
- net SCK: now also U$1.(PCINT4/T1/SCL/USCK/ADC4)PA4
- net VCC: no longer SV2.2, SV3.2, SV4.2, SV5.2
Changed lines of the file:
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@@
 <part name="SV4" library="con-lstb" deviceset="MA03-1" device=""/>
 <part name="SV5" library="con-lstb" deviceset="MA03-1" device=""/>
-<part name="P+2" library="supply1" deviceset="VCC" device=""/>
 <part name="GND2" library="supply1" deviceset="GND" device=""/>
 <part name="GND3" library="supply1" deviceset="GND" device=""/>
@@
 <part name="GND11" library="supply1" deviceset="GND" device=""/>
 <part name="R5" library="resistor" deviceset="R-EU_" device="R0805" value="3k9"/>
+<part name="P+9" library="supply1" deviceset="+5V" device=""/>
+<part name="P+2" library="supply1" deviceset="+5V" device=""/>
 </parts>
 <sheets>
@@
 <instance part="SV4" gate="G$1" x="228.6" y="48.26" rot="R90"/>
 <instance part="SV5" gate="G$1" x="243.84" y="48.26" rot="R90"/>
-<instance part="P+2" gate="VCC" x="256.54" y="68.58"/>
 <instance part="GND2" gate="1" x="256.54" y="43.18"/>
 <instance part="GND3" gate="1" x="187.96" y="58.42"/>
@@
 <instance part="GND11" gate="1" x="182.88" y="137.16"/>
 <instance part="R5" gate="G$1" x="96.52" y="45.72"/>
+<instance part="P+9" gate="1" x="251.46" y="172.72"/>
+<instance part="P+2" gate="1" x="256.54" y="71.12"/>
 </instances>
 <busses>
@@
 <net name="MOSI" class="0">
 <segment>
+<pinref part="RPI1" gate="RPI" pin="IO10/MOSI"/>
+<wire x1="210.82" y1="142.24" x2="195.58" y2="142.24" width="0.1524" layer="91"/>
+<label x="195.58" y="142.24" size="1.778" layer="95" rot="MR0"/>
+</segment>
+<segment>
+<pinref part="SV1" gate="G$1" pin="1"/>
+<wire x1="165.1" y1="154.94" x2="167.64" y2="154.94" width="0.1524" layer="91"/>
+<label x="167.64" y="154.94" size="1.778" layer="95"/>
+</segment>
+<segment>
 <pinref part="U$1" gate="G$1" pin="(PCINT6/OC1A/SDA/MOSI/ADC6)PA6"/>
 <wire x1="71.12" y1="144.78" x2="76.2" y2="144.78" width="0.1524" layer="91"/>
 <label x="76.2" y="144.78" size="1.778" layer="95"/>
-</segment>
-<segment>
-<pinref part="RPI1" gate="RPI" pin="IO10/MOSI"/>
-<wire x1="210.82" y1="142.24" x2="195.58" y2="142.24" width="0.1524" layer="91"/>
-<label x="195.58" y="142.24" size="1.778" layer="95" rot="MR0"/>
-</segment>
-<segment>
-<pinref part="SV1" gate="G$1" pin="1"/>
-<wire x1="165.1" y1="154.94" x2="167.64" y2="154.94" width="0.1524" layer="91"/>
-<label x="167.64" y="154.94" size="1.778" layer="95"/>
-</segment>
-</net>
-<net name="USCK" class="0">
-<segment>
-<pinref part="U$1" gate="G$1" pin="(PCINT4/T1/SCL/USCK/ADC4)PA4"/>
-<wire x1="71.12" y1="139.7" x2="76.2" y2="139.7" width="0.1524" layer="91"/>
-<label x="76.2" y="139.7" size="1.778" layer="95"/>
 </segment>
 </net>
@@
 <pinref part="U$1" gate="G$1" pin="VCC"/>
 <wire x1="15.24" y1="160.02" x2="20.32" y2="160.02" width="0.1524" layer="91"/>
-</segment>
-<segment>
-<pinref part="SV5" gate="G$1" pin="2"/>
-<wire x1="243.84" y1="55.88" x2="243.84" y2="63.5" width="0.1524" layer="91"/>
-<wire x1="243.84" y1="63.5" x2="256.54" y2="63.5" width="0.1524" layer="91"/>
-<pinref part="P+2" gate="VCC" pin="VCC"/>
-<wire x1="256.54" y1="63.5" x2="256.54" y2="66.04" width="0.1524" layer="91"/>
-<pinref part="SV2" gate="G$1" pin="2"/>
-<wire x1="198.12" y1="55.88" x2="198.12" y2="63.5" width="0.1524" layer="91"/>
-<wire x1="198.12" y1="63.5" x2="213.36" y2="63.5" width="0.1524" layer="91"/>
-<pinref part="SV3" gate="G$1" pin="2"/>
-<wire x1="213.36" y1="63.5" x2="228.6" y2="63.5" width="0.1524" layer="91"/>
-<wire x1="228.6" y1="63.5" x2="243.84" y2="63.5" width="0.1524" layer="91"/>
-<wire x1="213.36" y1="55.88" x2="213.36" y2="63.5" width="0.1524" layer="91"/>
-<pinref part="SV4" gate="G$1" pin="2"/>
-<wire x1="228.6" y1="55.88" x2="228.6" y2="63.5" width="0.1524" layer="91"/>
-<junction x="213.36" y="63.5"/>
-<junction x="228.6" y="63.5"/>
-<junction x="243.84" y="63.5"/>
 </segment>
 <segment>
@@
 <wire x1="76.2" y1="78.74" x2="86.36" y2="78.74" width="0.1524" layer="91"/>
 <wire x1="86.36" y1="78.74" x2="86.36" y2="83.82" width="0.1524" layer="91"/>
+<junction x="76.2" y="78.74"/>
 </segment>
 <segment>
@@
 <net name="MISO" class="0">
 <segment>
+<pinref part="RPI1" gate="RPI" pin="IO9/MISO"/>
+<wire x1="210.82" y1="139.7" x2="195.58" y2="139.7" width="0.1524" layer="91"/>
+<label x="195.58" y="139.7" size="1.778" layer="95" rot="MR0"/>
+</segment>
+<segment>
+<pinref part="SV1" gate="G$1" pin="9"/>
+<wire x1="165.1" y1="165.1" x2="167.64" y2="165.1" width="0.1524" layer="91"/>
+<label x="167.64" y="165.1" size="1.778" layer="95"/>
+</segment>
+<segment>
 <pinref part="U$1" gate="G$1" pin="(PCINT5/OC1B/MISO/DO/ADC5)PA5"/>
 <wire x1="71.12" y1="142.24" x2="76.2" y2="142.24" width="0.1524" layer="91"/>
 <label x="76.2" y="142.24" size="1.778" layer="95"/>
-</segment>
-<segment>
-<pinref part="RPI1" gate="RPI" pin="IO9/MISO"/>
-<wire x1="210.82" y1="139.7" x2="195.58" y2="139.7" width="0.1524" layer="91"/>
-<label x="195.58" y="139.7" size="1.778" layer="95" rot="MR0"/>
-</segment>
-<segment>
-<pinref part="SV1" gate="G$1" pin="9"/>
-<wire x1="165.1" y1="165.1" x2="167.64" y2="165.1" width="0.1524" layer="91"/>
-<label x="167.64" y="165.1" size="1.778" layer="95"/>
 </segment>
 </net>
@@
 <label x="83.82" y="165.1" size="1.778" layer="95" rot="R90"/>
 <pinref part="R1" gate="G$1" pin="1"/>
+<junction x="83.82" y="160.02"/>
 </segment>
 <segment>
@@
 <wire x1="165.1" y1="162.56" x2="167.64" y2="162.56" width="0.1524" layer="91"/>
 <label x="167.64" y="162.56" size="1.778" layer="95"/>
+</segment>
+<segment>
+<pinref part="U$1" gate="G$1" pin="(PCINT4/T1/SCL/USCK/ADC4)PA4"/>
+<wire x1="71.12" y1="139.7" x2="76.2" y2="139.7" width="0.1524" layer="91"/>
+<label x="76.2" y="139.7" size="1.778" layer="95"/>
 </segment>
 </net>
@@
 </segment>
 </net>
+<net name="+5V" class="0">
+<segment>
+<pinref part="RPI1" gate="RPI" pin="5V@1"/>
+<pinref part="P+9" gate="1" pin="+5V"/>
+<wire x1="246.38" y1="165.1" x2="251.46" y2="165.1" width="0.1524" layer="91"/>
+<wire x1="251.46" y1="165.1" x2="251.46" y2="170.18" width="0.1524" layer="91"/>
+</segment>
+<segment>
+<pinref part="SV5" gate="G$1" pin="2"/>
+<wire x1="243.84" y1="55.88" x2="243.84" y2="63.5" width="0.1524" layer="91"/>
+<wire x1="243.84" y1="63.5" x2="256.54" y2="63.5" width="0.1524" layer="91"/>
+<pinref part="SV2" gate="G$1" pin="2"/>
+<wire x1="198.12" y1="55.88" x2="198.12" y2="63.5" width="0.1524" layer="91"/>
+<wire x1="198.12" y1="63.5" x2="213.36" y2="63.5" width="0.1524" layer="91"/>
+<pinref part="SV3" gate="G$1" pin="2"/>
+<wire x1="213.36" y1="63.5" x2="228.6" y2="63.5" width="0.1524" layer="91"/>
+<wire x1="228.6" y1="63.5" x2="243.84" y2="63.5" width="0.1524" layer="91"/>
+<wire x1="213.36" y1="55.88" x2="213.36" y2="63.5" width="0.1524" layer="91"/>
+<pinref part="SV4" gate="G$1" pin="2"/>
+<wire x1="228.6" y1="55.88" x2="228.6" y2="63.5" width="0.1524" layer="91"/>
+<junction x="213.36" y="63.5"/>
+<junction x="228.6" y="63.5"/>
+<junction x="243.84" y="63.5"/>
+<pinref part="P+2" gate="1" pin="+5V"/>
+<wire x1="256.54" y1="63.5" x2="256.54" y2="68.58" width="0.1524" layer="91"/>
+</segment>
+</net>
